Commit message: Rename package from piklet_bot to piklet_description
- Updated package.xml with new package name
- Updated setup.py with new package name and entry points
- Updated setup.cfg with new script directories
- Updated all launch files to reference new package name
- Updated URDF/XACRO files to reference new package name
- Renamed directory structure: piklet_bot/ -> piklet_description/
- Renamed resource file: resource/piklet_bot -> resource/piklet_description
- Updated mesh file package references in bot_sample1.urdf

File: urdf/bot_sample1/bot_sample1.urdf (robot description, URDF)
Before this commit: robot piklet_bot, 4 links, 3 joints
Links:
- link arm_link: geometry collision cylinder length=0.4 radius=0.05; visual mesh filename=package://piklet_description/urdf/meshes/arm.dae
- link base_link: geometry collision box size=0.3 0.3 0.1; visual mesh filename=package://piklet_description/urdf/meshes/base.dae
- link gripper_link: geometry collision box size=0.1 0.05 0.05; visual mesh filename=package://piklet_description/urdf/meshes/gripper.dae

File: urdf/diffdrive_bot/diffdrive_bot.xacro (robot description, xacro)
@@ -1,5 +1,5 @@
 <?xml version="1.0"?>
 <robot name="diffdrive_robot" xmlns:xacro="http://ros.org/wiki/xacro">
-  <xacro:include filename="$(find piklet_bot)/urdf/diffdrive_robot_macro.xacro" />
+  <xacro:include filename="$(find piklet_description)/urdf/diffdrive_robot_macro.xacro" />
   <xacro:property name="base_radius" value="0.15" />
   <xacro:property name="passive_wheel_height" value="0.04" />

File: urdf/piklet_robot.urdf.xacro (robot description, xacro)
@@ -2,11 +2,11 @@
 <robot name="piklet_container_bot" xmlns:xacro="http://www.ros.org/wiki/xacro">
   <!-- Include modular parts -->
-  <xacro:include filename="$(find piklet_bot)/urdf/materials.xacro"/>
-  <xacro:include filename="$(find piklet_bot)/urdf/body.xacro"/>
-  <xacro:include filename="$(find piklet_bot)/urdf/wheel.xacro"/>
-  <xacro:include filename="$(find piklet_bot)/urdf/caster.xacro"/>
-  <xacro:include filename="$(find piklet_bot)/urdf/lidar.xacro"/>
-  <xacro:include filename="$(find piklet_bot)/urdf/depth_camera.xacro"/>
-  <xacro:include filename="$(find piklet_bot)/urdf/gazebo.xacro"/>
+  <xacro:include filename="$(find piklet_description)/urdf/materials.xacro"/>
+  <xacro:include filename="$(find piklet_description)/urdf/body.xacro"/>
+  <xacro:include filename="$(find piklet_description)/urdf/wheel.xacro"/>
+  <xacro:include filename="$(find piklet_description)/urdf/caster.xacro"/>
+  <xacro:include filename="$(find piklet_description)/urdf/lidar.xacro"/>
+  <xacro:include filename="$(find piklet_description)/urdf/depth_camera.xacro"/>
+  <xacro:include filename="$(find piklet_description)/urdf/gazebo.xacro"/>
   <!-- Base body (two plates + poles) -->
   <xacro:piklet_body parent="world"/>
