Commit message: feat(robot): complete arm with gripper and enable movement via built-in diffdrive
- Added full robotic arm with gripper to the URDF/Xacro
- Configured and tested differential drive for robot mobility
- Verified integrated motion of arm and base in simulation

File: urdf/arm-3-dof.xacro (robot description, xacro)
@@ -3,33 +3,23 @@
   <xacro:property name="M_PI" value="3.1415926535897931"/>
   <xacro:macro name="simple_arm" params="parent base_radius">
-    <link name="arm_base">
+    <link name="shoulder_yaw_link">
       <inertial>
-        <mass value="0.3"/>
-        <inertia ixx="5e-4" iyy="5e-4" izz="5e-4" ixy="0" ixz="0" iyz="0"/>
+        <mass value="1e-6"/>
+        <inertia ixx="1e-9" iyy="1e-9" izz="1e-9" ixy="0" ixz="0" iyz="0"/>
       </inertial>
-      <visual>
-        <geometry><cylinder radius="0.03" length="0.05"/></geometry>
-        <origin xyz="0 0 0.025" rpy="0 0 0"/>
-        <material name="blue"/>
-      </visual>
-      <collision>
-        <geometry><cylinder radius="0.03" length="0.05"/></geometry>
-        <origin xyz="0 0 0.025" rpy="0 0 0"/>
-      </collision>
     </link>
-    <joint name="arm_base_joint" type="fixed">
+    <joint name="shoulder_yaw" type="revolute">
       <parent link="${parent}"/>
-      <child link="arm_base"/>
-      <origin xyz="0 ${base_radius} 0.02" rpy="0 0 0"/>
-    </joint>
-    <link name="shoulder_yaw_link"/>
-    <joint name="shoulder_yaw" type="revolute">
-      <parent link="arm_base"/>
       <child link="shoulder_yaw_link"/>
-      <origin xyz="0 0 0.025" rpy="0 0 0"/>
+      <origin xyz="0 0 -0.05" rpy="0 0 0"/>
       <axis xyz="0 0 1"/>
       <limit lower="-1.57" upper="1.57" effort="5" velocity="1"/>
     </joint>
-    <link name="shoulder_pitch_link"/>
+    <link name="shoulder_pitch_link">
+      <inertial>
+        <mass value="1e-6"/>
+        <inertia ixx="1e-9" iyy="1e-9" izz="1e-9" ixy="0" ixz="0" iyz="0"/>
+      </inertial>
+    </link>
     <joint name="shoulder_pitch" type="revolute">
       <parent link="shoulder_yaw_link"/>
@@ -39,5 +29,10 @@
       <limit lower="-1.57" upper="1.57" effort="5" velocity="1"/>
     </joint>
-    <link name="shoulder_roll_link"/>
+    <link name="shoulder_roll_link">
+      <inertial>
+        <mass value="1e-6"/>
+        <inertia ixx="1e-9" iyy="1e-9" izz="1e-9" ixy="0" ixz="0" iyz="0"/>
+      </inertial>
+    </link>
     <joint name="shoulder_roll" type="revolute">
       <parent link="shoulder_pitch_link"/>
@@ -89,5 +84,5 @@
       <limit lower="-1.57" upper="1.57" effort="5" velocity="1"/>
     </joint>
-    <link name="arm_link3">
+    <link name="arm_link_end">
       <inertial>
         <mass value="0.15"/>
@@ -106,5 +101,5 @@
     <joint name="wrist_joint" type="revolute">
       <parent link="arm_link2"/>
-      <child link="arm_link3"/>
+      <child link="arm_link_end"/>
       <origin xyz="0.12 0 0" rpy="0 0 0"/>
       <axis xyz="0 1 0"/>

File: urdf/body.xacro (robot description, xacro)
@@ -10,8 +10,7 @@
     <link name="base_link">
       <inertial>
-        <inertia ixx="1.0" ixy="0.0" ixz="0.0" iyy="1.0" iyz="0.0" izz="1.0"/>
         <mass value="5" />
         <origin xyz="0 0 0" />
-        <cylinder_inertia m="5" r="${base_radius}" h="0.02" />
+        <xacro:cylinder_inertia m="5" r="${base_radius}" h="0.02" />
       </inertial>
       <visual>
@@ -32,8 +31,7 @@
     <link name="base_top">
       <inertial>
-        <inertia ixx="1.0" ixy="0.0" ixz="0.0" iyy="1.0" iyz="0.0" izz="1.0"/>
         <mass value="5" />
         <origin xyz="0 0 0" />
-        <cylinder_inertia m="5" r="${base_radius}" h="0.02" />
+        <xacro:cylinder_inertia m="5" r="${base_radius}" h="0.02" />
       </inertial>
       <visual>
@@ -76,3 +74,25 @@
     </joint>
   </xacro:macro>
+  <!-- front mount -->
+  <link name="front_mount">
+    <inertial>
+      <mass value="0.3" />
+      <origin xyz="0 0 0" />
+      <xacro:cylinder_inertia m="0.3" r="0.03" h="${front_mount_length}" />
+    </inertial>
+    <visual>
+      <geometry><cylinder radius="0.03" length="${front_mount_length}"/></geometry>
+      <origin xyz="0 0 0" rpy="0 0 0"/>
+      <material name="blue"/>
+    </visual>
+    <collision>
+      <geometry><cylinder radius="0.03" length="${front_mount_length}"/></geometry>
+      <origin xyz="0 0 0" rpy="0 0 0"/>
+    </collision>
+  </link>
+  <joint name="front_mount_joint" type="fixed">
+    <parent link="base_top"/>
+    <child link="front_mount"/>
+    <origin xyz="0.13 0 0.09" rpy="0 0 0"/>
+  </joint>
 </robot>

File: urdf/depth_camera.xacro (robot description, xacro)
@@ -8,8 +8,8 @@
       </visual>
     </link>
-    <joint name="depth_camera_joint" type="fixed">
-      <origin xyz="${xyz}"/>
+    <joint name="depth_camera_mount" type="fixed">
       <parent link="${parent}"/>
       <child link="depth_camera_link"/>
+      <origin xyz="${xyz}" />
     </joint>
   </xacro:macro>

File: urdf/gazebo.xacro (robot description, xacro)
@@ -6,14 +6,8 @@
   <xacro:macro name="diff_drive_plugin" params="left right">
     <gazebo>
-      <plugin name="diff_drive" filename="gz-sim-diff-drive-system">
+      <plugin name="gz::sim::systems::DiffDrive" filename="gz-sim-diff-drive-system">
         <!-- wheels -->
         <left_joint>${left}</left_joint>
         <right_joint>${right}</right_joint>
-        <!-- topic interface -->
-        <ros>
-          <namespace>/piklet_bot</namespace>
-          <topic name="cmd_vel" type="geometry_msgs/msg/Twist"/>
-          <topic name="odom" type="nav_msgs/msg/Odometry"/>
-        </ros>
         <!-- physics -->
         <wheel_separation>0.34</wheel_separation>
@@ -23,4 +17,11 @@
         <base_frame>base_link</base_frame>
         <publish_odom>true</publish_odom>
+        <!-- topic interface -->
+        <topic>cmd_vel</topic>
+      </plugin>
+      <plugin filename="gz-sim-joint-state-publisher-system" name="gz::sim::systems::JointStatePublisher">
+        <topic>joint_states</topic>
+        <joint_name>right_wheel_joint</joint_name>
+        <joint_name>left_wheel_joint</joint_name>
       </plugin>
     </gazebo>
@@ -47,5 +48,5 @@
           </range>
         </ray>
-        <plugin name="lidar_ros" filename="gz-sim-ros2-laser-scan">
+        <plugin name="lidar_ros" filename="gz-sim-ros2-generic-sensor-system">
           <ros>
             <topic name="scan" type="sensor_msgs/msg/LaserScan"/>
@@ -73,5 +74,5 @@
           </clip>
         </camera>
-        <plugin name="depth_camera_ros" filename="gz-sim-ros2-camera">
+        <plugin name="camera_ros" filename="gz-sim-ros2-generic-sensor-system">
           <ros>
             <topic name="image_raw" type="sensor_msgs/msg/Image"/>

File: urdf/materials.xacro (robot description, xacro)
@@ -12,4 +12,5 @@
   <xacro:color_material name="darkgray" r="0.3" g="0.3" b="0.3" a="1"/>
   <xacro:color_material name="red" r="0.8" g="0.1" b="0.1" a="1"/>
+  <xacro:color_material name="yellow" r="0.5" g="0.3" b="0.1" a="1"/>
   <xacro:color_material name="green" r="0.2" g="0.8" b="0.2" a="1"/>
   <xacro:color_material name="white" r="1" g="1" b="1" a="1"/>

File: urdf/piklet_robot.urdf.xacro (robot description, xacro)
@@ -10,4 +10,5 @@
   <xacro:property name="wheel_mass" value="2.5" />
   <xacro:property name="pole_length" value="0.2" />
+  <xacro:property name="front_mount_length" value="0.2" />
   <!-- Include modular parts -->
   <xacro:include filename="$(find piklet_description)/urdf/materials.xacro"/>
@@ -19,4 +20,5 @@
   <xacro:include filename="$(find piklet_description)/urdf/gazebo.xacro"/>
   <xacro:include filename="$(find piklet_description)/urdf/arm-3-dof.xacro"/>
+  <xacro:include filename="$(find piklet_description)/urdf/finger-2-gripper.xacro"/>
   <!-- Base body (two plates + poles) -->
   <xacro:piklet_body parent="world"/>
@@ -43,12 +45,15 @@
     <origin xyz="0.02 0.02 0 " rpy="${M_PI/2} 0 0" />
   </xacro:passive_wheel_link>
-  <!-- Arm -->
-  <xacro:simple_arm parent="base_top" base_radius="${base_radius}"/>
+  <!-- Arm attaches to mount lower part -->
+  <xacro:simple_arm parent="front_mount" base_radius="${base_radius}"/>
+  <!-- 2 finger parallel gripper -->
+  <xacro:parallel_gripper parent_link="arm_link_end" xyz="0.1 0 0"/>
   <!-- Sensors -->
   <xacro:lidar_sensor parent="base_top" xyz="0 0 0.030"/>
-  <xacro:depth_camera parent="base_top" xyz="0.13 0 0.025"/>
+  <!-- Camera attaches on top of mount -->
+  <xacro:depth_camera parent="front_mount" xyz="0 0 0.12"/>
   <!-- Gazebo Plugins -->
   <xacro:diff_drive_plugin left="left_wheel_joint" right="right_wheel_joint"/>
-  <xacro:lidar_plugin parent="lidar_link"/>
-  <xacro:depth_camera_plugin parent="depth_camera_link"/>
+  <!--xacro:lidar_plugin parent="lidar_link"/-->
+  <!--xacro:depth_camera_plugin parent="depth_camera_link"/-->
 </robot>

File: urdf/wheel.xacro (robot description, xacro)
@@ -33,18 +33,34 @@
     </joint>
   </xacro:macro>
-  <xacro:macro name="drive_wheel" params="name parent xyz">
+  <xacro:macro name="passive_wheel_joint" params="name parent child *origin">
+    <joint name="${name}" type="fixed" >
+      <parent link="${parent}" />
+      <child link="${child}" />
+      <xacro:insert_block name="origin" />
+    </joint>
+  </xacro:macro>
+  <xacro:macro name="passive_wheel_link" params="name *origin">
     <link name="${name}">
       <visual>
-        <geometry><cylinder radius="0.05" length="0.02"/></geometry>
-        <origin rpy="0 1.57 0"/>
-        <material name="black"/>
+        <xacro:insert_block name="origin"/>
+        <geometry>
+          <sphere radius="${passive_wheel_radius}" />
+        </geometry>
+        <material name="Black" />
       </visual>
+      <collision>
+        <geometry>
+          <sphere radius="${passive_wheel_radius}" />
+        </geometry>
+        <origin xyz="0 0.02 0" rpy="${M_PI/2} 0 0" />
+      </collision>
+      <inertial>
+        <mass value="${passive_wheel_mass}" />
+        <origin xyz="0 0 0" />
+        <inertia ixx="0.001" ixy="0.0" ixz="0.0"
+          iyy="0.001" iyz="0.0"
+          izz="0.001" />
+      </inertial>
     </link>
-    <joint name="${name}_joint" type="continuous">
-      <origin xyz="${xyz}" rpy="0 1.57 0"/>
-      <parent link="${parent}"/>
-      <child link="${name}"/>
-      <axis xyz="0 0 1"/>
-    </joint>
   </xacro:macro>
 </robot>
