Commit message: update robot model design

File: urdf/body.xacro (robot description, xacro)
@@ -1,29 +1,63 @@
 <?xml version="1.0"?>
 <robot xmlns:xacro="http://www.ros.org/wiki/xacro">
+  <xacro:macro name="cylinder_inertia" params="m r h">
+    <inertia ixx="${m*(3*r*r+h*h)/12}" ixy="0" ixz="0"
+      iyy="${m*(3*r*r+h*h)/12}" iyz="0"
+      izz="${m*(3*r*r+h*h)/12}" />
+  </xacro:macro>
   <xacro:macro name="piklet_body" params="parent">
     <!-- Bottom plate -->
-    <link name="base_bottom">
+    <link name="base_link">
+      <inertial>
+        <inertia ixx="1.0" ixy="0.0" ixz="0.0" iyy="1.0" iyz="0.0" izz="1.0"/>
+        <mass value="5" />
+        <origin xyz="0 0 0" />
+        <cylinder_inertia m="5" r="${base_radius}" h="0.02" />
+      </inertial>
       <visual>
-        <geometry><box size="0.4 0.3 0.02"/></geometry>
-        <material name="gray"/>
+        <origin xyz="0 0 0" rpy="0 0 0" />
+          <cylinder length="0.02" radius="${base_radius}" />
+        </geometry>
+        <material name="white" />
       </visual>
+      <collision>
+        <origin xyz="0 0 0" rpy="0 0 0" />
+        <geometry>
+          <cylinder length="0.02" radius="${base_radius}" />
+        </geometry>
+      </collision>
     </link>
     <!-- Top plate -->
     <link name="base_top">
+      <inertial>
+        <inertia ixx="1.0" ixy="0.0" ixz="0.0" iyy="1.0" iyz="0.0" izz="1.0"/>
+        <mass value="5" />
+        <origin xyz="0 0 0" />
+        <cylinder_inertia m="5" r="${base_radius}" h="0.02" />
+      </inertial>
       <visual>
-        <geometry><box size="0.4 0.3 0.02"/></geometry>
-        <material name="blue"/>
+        <origin xyz="0 0 0" rpy="0 0 0" />
+        <geometry>
+          <cylinder length="0.02" radius="${base_radius}" />
+        </geometry>
+        <material name="white" />
       </visual>
+      <collision>
+        <origin xyz="0 0 0" rpy="0 0 0" />
+        <geometry>
+          <cylinder length="0.02" radius="${base_radius}" />
+        </geometry>
+      </collision>
     </link>
     <joint name="base_top_joint" type="fixed">
       <origin xyz="0 0 0.2"/>
-      <parent link="base_bottom"/>
+      <parent link="base_link"/>
       <child link="base_top"/>
     </joint>
     <!-- Poles -->
-    <xacro:pole name="pole_fl" xyz="0.18 0.13 0.1"/>
-    <xacro:pole name="pole_fr" xyz="0.18 -0.13 0.1"/>
-    <xacro:pole name="pole_bl" xyz="-0.18 0.13 0.1"/>
-    <xacro:pole name="pole_br" xyz="-0.18 -0.13 0.1"/>
+    <xacro:pole name="pole_fl" xyz="0.1 0.1 0.1"/>
+    <xacro:pole name="pole_fr" xyz="0.1 -0.1 0.1"/>
+    <xacro:pole name="pole_bl" xyz="-0.1 0.1 0.1"/>
+    <xacro:pole name="pole_br" xyz="-0.1 -0.1 0.1"/>
   </xacro:macro>
   <!-- Pole macro -->
@@ -31,5 +65,5 @@
     <link name="${name}">
       <visual>
-        <geometry><cylinder radius="0.01" length="0.2"/></geometry>
+        <geometry><cylinder radius="0.01" length="${pole_length}"/></geometry>
         <material name="darkgray"/>
       </visual>
@@ -37,5 +71,5 @@
     <joint name="${name}_joint" type="fixed">
       <origin xyz="${xyz}" rpy="0 0 0"/>
-      <parent link="base_bottom"/>
+      <parent link="base_link"/>
       <child link="${name}"/>
     </joint>

File: urdf/caster.xacro (robot description, xacro)
@@ -1,16 +1,34 @@
 <?xml version="1.0"?>
 <robot xmlns:xacro="http://www.ros.org/wiki/xacro">
-  <xacro:macro name="caster_wheel" params="name parent xyz">
+  <xacro:macro name="passive_wheel_joint" params="name parent child *origin">
+    <joint name="${name}" type="fixed" >
+      <parent link="${parent}" />
+      <child link="${child}" />
+      <xacro:insert_block name="origin" />
+    </joint>
+  </xacro:macro>
+  <xacro:macro name="passive_wheel_link" params="name *origin">
     <link name="${name}">
       <visual>
-        <geometry><sphere radius="0.025"/></geometry>
-        <material name="darkgray"/>
+        <xacro:insert_block name="origin"/>
+        <geometry>
+          <sphere radius="${passive_wheel_radius}" />
+        </geometry>
+        <material name="black" />
       </visual>
+      <collision>
+        <geometry>
+          <sphere radius="${passive_wheel_radius}" />
+        </geometry>
+        <origin xyz="0 0.02 0" rpy="${M_PI/2} 0 0" />
+      </collision>
+      <inertial>
+        <mass value="${passive_wheel_mass}" />
+        <origin xyz="0 0 0" />
+        <inertia ixx="0.001" ixy="0.0" ixz="0.0"
+          iyy="0.001" iyz="0.0"
+          izz="0.001" />
+      </inertial>
     </link>
-    <joint name="${name}_joint" type="fixed">
-      <origin xyz="${xyz}"/>
-      <parent link="${parent}"/>
-      <child link="${name}"/>
-    </joint>
   </xacro:macro>
 </robot>

File: urdf/lidar.xacro (robot description, xacro)
@@ -5,5 +5,5 @@
       <visual>
         <geometry><cylinder radius="0.04" length="0.05"/></geometry>
-        <origin xyz="0 0 0.025"/>
+        <origin xyz="0 0 0"/>
         <material name="red"/>
       </visual>

File: urdf/materials.xacro (robot description, xacro)
@@ -13,3 +13,4 @@
   <xacro:color_material name="red" r="0.8" g="0.1" b="0.1" a="1"/>
   <xacro:color_material name="green" r="0.2" g="0.8" b="0.2" a="1"/>
+  <xacro:color_material name="white" r="1" g="1" b="1" a="1"/>
 </robot>

File: urdf/piklet_robot.urdf.xacro (robot description, xacro)
@@ -1,4 +1,13 @@
 <?xml version="1.0"?>
 <robot name="piklet_container_bot" xmlns:xacro="http://www.ros.org/wiki/xacro">
+  <xacro:property name="M_PI" value="3.1415926535897931" />
+  <xacro:property name="base_radius" value="0.15" />
+  <xacro:property name="passive_wheel_height" value="0.04" />
+  <xacro:property name="passive_wheel_radius" value="0.025" />
+  <xacro:property name="passive_wheel_mass" value="0.5" />
+  <xacro:property name="wheel_radius" value="0.039" />
+  <xacro:property name="wheel_height" value="0.02" />
+  <xacro:property name="wheel_mass" value="2.5" />
+  <xacro:property name="pole_length" value="0.2" />
   <!-- Include modular parts -->
   <xacro:include filename="$(find piklet_description)/urdf/materials.xacro"/>
@@ -12,12 +21,28 @@
   <xacro:piklet_body parent="world"/>
   <!-- Drive wheels -->
-  <xacro:drive_wheel name="left_wheel"  parent="base_bottom" xyz="0 -0.17 0.05"/>
-  <xacro:drive_wheel name="right_wheel" parent="base_bottom" xyz="0 0.17 0.05"/>
+  <xacro:wheel side="right" parent="base_link" translateX="0"
+    translateY="-${base_radius}"/>
+  <xacro:wheel side="left" parent="base_link" translateX="0"
+    translateY="${base_radius}" />
   <!-- Casters -->
-  <xacro:caster_wheel name="caster_front" parent="base_bottom" xyz="0.15 0 0.02"/>
-  <xacro:caster_wheel name="caster_back"  parent="base_bottom" xyz="-0.15 0 0.02"/>
+  <xacro:passive_wheel_joint name="passive_wheel_front_joint"
+    parent="base_link"
+    child="passive_wheel_front_link">
+  <origin xyz="0.115 0.0 0.007" rpy="${-M_PI/2} 0 0" />
+  </xacro:passive_wheel_joint>
+  <xacro:passive_wheel_link name="passive_wheel_front_link">
+    <origin xyz="0 0.02 0" rpy="${M_PI/2} 0 0" />
+  </xacro:passive_wheel_link>
+  <xacro:passive_wheel_joint name="passive_wheel_back_joint"
+    parent="base_link"
+    child="passive_wheel_back_link">
+    <origin xyz="-0.135 0.0 0.009" rpy="${-M_PI/2} 0 0"/>
+  </xacro:passive_wheel_joint>
+  <xacro:passive_wheel_link name="passive_wheel_back_link">
+    <origin xyz="0.02 0.02 0 " rpy="${M_PI/2} 0 0" />
+  </xacro:passive_wheel_link>
   <!-- Sensors -->
-  <xacro:lidar_sensor parent="base_top" xyz="0 0 0.02"/>
-  <xacro:depth_camera parent="base_top" xyz="0.2 0 0.02"/>
+  <xacro:lidar_sensor parent="base_top" xyz="0 0 0.030"/>
+  <xacro:depth_camera parent="base_top" xyz="0.13 0 0.025"/>
   <!-- Gazebo Plugins -->
   <xacro:diff_drive_plugin left="left_wheel_joint" right="right_wheel_joint"/>

File: urdf/wheel.xacro (robot description, xacro)
@@ -1,4 +1,36 @@
 <?xml version="1.0"?>
 <robot xmlns:xacro="http://www.ros.org/wiki/xacro">
+  <xacro:macro name="wheel" params="side parent translateX translateY">
+    <link name="${side}_wheel">
+      <visual>
+        <origin xyz="0 0 0" rpy="${M_PI/2} 0 0" />
+        <geometry>
+          <cylinder length="${wheel_height}" radius="${wheel_radius}" />
+        </geometry>
+        <material name="black" />
+      </visual>
+      <collision>
+        <origin xyz="0 0 0" rpy="${M_PI/2} 0 0 " />
+        <geometry>
+          <cylinder length="${wheel_height}" radius="${wheel_radius}" />
+        </geometry>
+      </collision>
+      <inertial>
+        <mass value="${wheel_mass}" />
+        <origin xyz="0 0 0" />
+        <inertia ixx="0.001" ixy="0.0" ixz="0.0"
+          iyy="0.001" iyz="0.0"
+          izz="0.001" />
+      </inertial>
+    </link>
+    <joint name="${side}_wheel_joint" type="continuous">
+      <parent link="${parent}" />
+      <child link="${side}_wheel" />
+      <origin xyz="0 ${translateY} 0" rpy="0 0 0" />
+      <axis xyz="0 1 0" rpy="0 0 0" />
+      <limit effort="100" velocity="100" />
+      <joint_properties damping="0.0" friction="0.0" />
+    </joint>
+  </xacro:macro>
   <xacro:macro name="drive_wheel" params="name parent xyz">
     <link name="${name}">

Commit message: Add 3-DOF shoulder arm with elbow and wrist

File: urdf/body.xacro (robot description, xacro)
@@ -17,4 +17,5 @@
       <visual>
         <origin xyz="0 0 0" rpy="0 0 0" />
+        <geometry>
           <cylinder length="0.02" radius="${base_radius}" />
         </geometry>

File: urdf/gazebo.xacro (robot description, xacro)
@@ -21,5 +21,5 @@
         <!-- odom frame -->
         <odom_frame>odom</odom_frame>
-        <base_frame>base_bottom</base_frame>
+        <base_frame>base_link</base_frame>
         <publish_odom>true</publish_odom>
       </plugin>

File: urdf/piklet_robot.urdf.xacro (robot description, xacro)
@@ -18,4 +18,5 @@
   <xacro:include filename="$(find piklet_description)/urdf/depth_camera.xacro"/>
   <xacro:include filename="$(find piklet_description)/urdf/gazebo.xacro"/>
+  <xacro:include filename="$(find piklet_description)/urdf/arm-3-dof.xacro"/>
   <!-- Base body (two plates + poles) -->
   <xacro:piklet_body parent="world"/>
@@ -42,4 +43,6 @@
     <origin xyz="0.02 0.02 0 " rpy="${M_PI/2} 0 0" />
   </xacro:passive_wheel_link>
+  <!-- Arm -->
+  <xacro:simple_arm parent="base_top" base_radius="${base_radius}"/>
   <!-- Sensors -->
   <xacro:lidar_sensor parent="base_top" xyz="0 0 0.030"/>

Commit message: add minor fixes in xacro/urdf files

File: urdf/body.xacro (robot description, xacro)
@@ -7,4 +7,11 @@
   </xacro:macro>
   <xacro:macro name="piklet_body" params="parent">
+    <link name="base_footprint" />
+    <!-- The base footprint of the robot is located underneath the chassis -->
+    <joint name="base_joint" type="fixed">
+      <parent link="base_footprint"/>
+      <child link="base_link" />
+      <origin xyz="0 0 0.1" rpy="0 0 0"/>
+    </joint>
     <!-- Bottom plate -->
     <link name="base_link">
@@ -67,4 +74,10 @@
         <material name="darkgray"/>
       </visual>
+      <collision>
+        <origin xyz="0 0 0" rpy="0 0 0" />
+        <geometry>
+          <cylinder length="${pole_length}" radius="0.01" />
+        </geometry>
+      </collision>
     </link>
     <joint name="${name}_joint" type="fixed">

File: urdf/depth_camera.xacro (robot description, xacro)
@@ -7,4 +7,10 @@
         <material name="green"/>
       </visual>
+      <collision>
+        <origin xyz="0 0 0" rpy="0 0 0" />
+        <geometry>
+          <box size="0.06 0.04 0.04" />
+        </geometry>
+      </collision>
     </link>
     <joint name="depth_camera_mount" type="fixed">

File: urdf/gazebo.xacro (robot description, xacro)
@@ -13,4 +13,6 @@
         <wheel_separation>0.34</wheel_separation>
         <wheel_radius>0.05</wheel_radius>
+        <max_wheel_torque>10.0</max_wheel_torque>
+        <max_wheel_acceleration>5.0</max_wheel_acceleration>
         <!-- odom frame -->
         <odom_frame>odom</odom_frame>
@@ -19,4 +21,6 @@
         <!-- topic interface -->
         <topic>cmd_vel</topic>
+        <!-- stop wheels if no command received -->
+        <command_timeout>0.5</command_timeout> <!-- seconds -->
       </plugin>
       <plugin filename="gz-sim-joint-state-publisher-system" name="gz::sim::systems::JointStatePublisher">

File: urdf/lidar.xacro (robot description, xacro)
@@ -8,4 +8,10 @@
         <material name="red"/>
       </visual>
+      <collision>
+        <origin xyz="0 0 0" rpy="0 0 0" />
+        <geometry>
+          <cylinder length="0.05" radius="0.04" />
+        </geometry>
+      </collision>
     </link>
     <joint name="lidar_joint" type="fixed">

File: urdf/piklet_robot.urdf.xacro (robot description, xacro)
@@ -6,5 +6,5 @@
   <xacro:property name="passive_wheel_radius" value="0.025" />
   <xacro:property name="passive_wheel_mass" value="0.5" />
-  <xacro:property name="wheel_radius" value="0.039" />
+  <xacro:property name="wheel_radius" value="0.04" />
   <xacro:property name="wheel_height" value="0.02" />
   <xacro:property name="wheel_mass" value="2.5" />
@@ -55,5 +55,5 @@
   <!-- Gazebo Plugins -->
   <xacro:diff_drive_plugin left="left_wheel_joint" right="right_wheel_joint"/>
-  <!--xacro:lidar_plugin parent="lidar_link"/-->
-  <!--xacro:depth_camera_plugin parent="depth_camera_link"/-->
+  <xacro:lidar_plugin parent="lidar_link"/>
+  <xacro:depth_camera_plugin parent="depth_camera_link"/>
 </robot>

File: urdf/wheel.xacro (robot description, xacro)
@@ -15,4 +15,12 @@
           <cylinder length="${wheel_height}" radius="${wheel_radius}" />
         </geometry>
+        <surface>
+          <friction>
+            <ode>
+              <mu>1.0</mu>
+              <mu2>1.0</mu2>
+            </ode>
+          </friction>
+        </surface>
       </collision>
       <inertial>
@@ -30,5 +38,5 @@
       <axis xyz="0 1 0" rpy="0 0 0" />
       <limit effort="100" velocity="100" />
-      <joint_properties damping="0.0" friction="0.0" />
+      <dynamics damping="0.5" friction="0.2"/>
     </joint>
   </xacro:macro>

Commit message: add ros_control settings

File: urdf/body.xacro (robot description, xacro)
@@ -7,8 +7,6 @@
   </xacro:macro>
   <xacro:macro name="piklet_body" params="parent">
-    <link name="base_footprint" />
-    <!-- The base footprint of the robot is located underneath the chassis -->
     <joint name="base_joint" type="fixed">
-      <parent link="base_footprint"/>
+      <parent link="${parent}"/>
       <child link="base_link" />
       <origin xyz="0 0 0.1" rpy="0 0 0"/>

File: urdf/piklet_robot.urdf.xacro (robot description, xacro)
@@ -1,4 +1,5 @@
 <?xml version="1.0"?>
 <robot name="piklet_container_bot" xmlns:xacro="http://www.ros.org/wiki/xacro">
+  <xacro:arg name="prefix" default="" />
   <xacro:property name="M_PI" value="3.1415926535897931" />
   <xacro:property name="base_radius" value="0.15" />
@@ -21,6 +22,9 @@
   <xacro:include filename="$(find piklet_description)/urdf/arm-3-dof.xacro"/>
   <xacro:include filename="$(find piklet_description)/urdf/finger-2-gripper.xacro"/>
+  <xacro:include filename="$(find piklet_description)/urdf/piklet_ros2_control.xacro"/>
   <!-- Base body (two plates + poles) -->
-  <xacro:piklet_body parent="world"/>
+  <!-- The base footprint of the robot is located underneath the chassis -->
+  <link name="base_footprint" />
+  <xacro:piklet_body parent="base_footprint"/>
   <!-- Drive wheels -->
   <xacro:wheel side="right" parent="base_link" translateX="0"
@@ -54,6 +58,7 @@
   <xacro:depth_camera parent="front_mount" xyz="0 0 0.12"/>
   <!-- Gazebo Plugins -->
-  <xacro:diff_drive_plugin left="left_wheel_joint" right="right_wheel_joint"/>
   <xacro:lidar_plugin parent="lidar_link"/>
   <xacro:depth_camera_plugin parent="depth_camera_link"/>
+  <!-- ros2_control -->
+  <xacro:piklet_diffdrive_ros2_control name="Piklet" prefix="$(arg prefix)" />
 </robot>
