Commit message: add test

File: urdf/piklet_m1/piklet_robot.urdf.xacro (robot description, xacro)
@@ -1,4 +1,4 @@
 <?xml version="1.0"?>
-<robot name="piklet_container_bot" xmlns:xacro="http://www.ros.org/wiki/xacro">
+<robot name="piklet_m1" xmlns:xacro="http://www.ros.org/wiki/xacro">
   <xacro:arg name="prefix" default="" />
   <xacro:property name="M_PI" value="3.1415926535897931" />
@@ -12,15 +12,16 @@
   <xacro:property name="pole_length" value="0.2" />
   <xacro:property name="front_mount_length" value="0.2" />
+  <xacro:property name="robot_path" value="$(find piklet_description)/urdf/piklet_m1" />
   <!-- Include modular parts -->
-  <xacro:include filename="$(find piklet_description)/urdf/materials.xacro"/>
-  <xacro:include filename="$(find piklet_description)/urdf/body.xacro"/>
-  <xacro:include filename="$(find piklet_description)/urdf/wheel.xacro"/>
-  <xacro:include filename="$(find piklet_description)/urdf/caster.xacro"/>
-  <xacro:include filename="$(find piklet_description)/urdf/lidar.xacro"/>
-  <xacro:include filename="$(find piklet_description)/urdf/depth_camera.xacro"/>
-  <xacro:include filename="$(find piklet_description)/urdf/gazebo.xacro"/>
-  <xacro:include filename="$(find piklet_description)/urdf/arm-3-dof.xacro"/>
-  <xacro:include filename="$(find piklet_description)/urdf/finger-2-gripper.xacro"/>
-  <xacro:include filename="$(find piklet_description)/urdf/piklet_ros2_control.xacro"/>
+  <xacro:include filename="${robot_path}/materials.xacro"/>
+  <xacro:include filename="${robot_path}/body.xacro"/>
+  <xacro:include filename="${robot_path}/wheel.xacro"/>
+  <xacro:include filename="${robot_path}/caster.xacro"/>
+  <xacro:include filename="${robot_path}/lidar.xacro"/>
+  <xacro:include filename="${robot_path}/depth_camera.xacro"/>
+  <xacro:include filename="${robot_path}/gazebo.xacro"/>
+  <xacro:include filename="${robot_path}/arm-3-dof.xacro"/>
+  <xacro:include filename="${robot_path}/finger-2-gripper.xacro"/>
+  <xacro:include filename="${robot_path}/piklet_ros2_control.xacro"/>
   <!-- Base body (two plates + poles) -->
   <!-- The base footprint of the robot is located underneath the chassis -->
