Commit message: use ros2_control to publish /joint_states
* additional settings to visualize links in rviz when
ros2_control joint_state_broadcaster is used

File: urdf/piklet_m1/arm-3-dof.xacro (robot description, xacro)
@@ -4,4 +4,9 @@
   <xacro:macro name="simple_arm" params="parent base_radius">
     <link name="shoulder_yaw_link">
+      <visual>
+        <geometry>
+          <sphere radius="0.01"/>
+        </geometry>
+      </visual>
       <inertial>
         <mass value="1e-6"/>
@@ -17,4 +22,9 @@
     </joint>
     <link name="shoulder_pitch_link">
+      <visual>
+        <geometry>
+          <sphere radius="0.01"/>
+        </geometry>
+      </visual>
       <inertial>
         <mass value="1e-6"/>
@@ -30,4 +40,9 @@
     </joint>
     <link name="shoulder_roll_link">
+      <visual>
+        <geometry>
+          <sphere radius="0.01"/>
+        </geometry>
+      </visual>
       <inertial>
         <mass value="1e-6"/>

File: urdf/piklet_m1/piklet_robot.urdf.xacro (robot description, xacro)
@@ -26,6 +26,6 @@
   <!-- Base body (two plates + poles) -->
   <!-- The base footprint of the robot is located underneath the chassis -->
-  <link name="base_footprint" />
-  <xacro:piklet_body parent="base_footprint"/>
+  <link name="world" />
+  <xacro:piklet_body parent="world"/>
   <!-- Drive wheels -->
   <xacro:wheel side="right" parent="base_link" translateX="0"
@@ -50,5 +50,5 @@
     <origin xyz="0.02 0.02 0 " rpy="${M_PI/2} 0 0" />
   </xacro:passive_wheel_link>
-  <!-- Arm attaches to mount lower part -->
+  <!-- Arm attaches to front_mount lower part -->
   <xacro:simple_arm parent="front_mount" base_radius="${base_radius}"/>
   <!-- 2 finger parallel gripper -->
@@ -62,4 +62,4 @@
   <xacro:depth_camera_plugin parent="depth_camera_link"/>
   <!-- ros2_control -->
-  <xacro:piklet_diffdrive_ros2_control name="Piklet" prefix="$(arg prefix)" />
+  <xacro:piklet_diffdrive_ros2_control name="Piklet_m1" prefix="$(arg prefix)" />
 </robot>

File: urdf/piklet_m1/piklet_ros2_control.xacro (robot description, xacro)
@@ -3,4 +3,7 @@
   <xacro:macro name="piklet_diffdrive_ros2_control" params="name prefix">
     <ros2_control name="${name}" type="system">
+      <hardware>
+        <plugin>mock_components/GenericSystem</plugin>
+      </hardware>
       <joint name="${prefix}left_wheel_joint">
         <command_interface name="velocity"/>
@@ -13,4 +16,24 @@
         <state_interface name="velocity"/>
       </joint>
+      <joint name="shoulder_yaw">
+        <command_interface name="position"/>
+        <state_interface name="position"/>
+      </joint>
+      <joint name="shoulder_roll">
+        <command_interface name="position"/>
+        <state_interface name="position"/>
+      </joint>
+      <joint name="shoulder_pitch">
+        <command_interface name="position"/>
+        <state_interface name="position"/>
+      </joint>
+      <joint name="elbow_joint">
+        <command_interface name="position"/>
+        <state_interface name="position"/>
+      </joint>
+      <joint name="wrist_joint">
+        <command_interface name="position"/>
+        <state_interface name="position"/>
+      </joint>
     </ros2_control>
   </xacro:macro>
